File: lipo_disconnector.kicad_sch (KiCad schematic)
At the start: 3 parts

Commit message: update
Parts:
- added H1, H2, H_GND: MountingHole_Pad, MountingHole:MountingHole_4mm_Pad, symbol Mechanical:MountingHole_Pad
- added P1, P2, P_GND: Conn_01x01_Male, Connector_PinHeader_2.54mm:PinHeader_1x01_P2.54mm_Vertical, symbol Connector:Conn_01x01_Male
- J1: renamed from U; value (none) -> Conn_Batt1; footprint (none) -> Connector_JST:JST_PH_S2B-PH-SM4-TB_1x02-1MP_P2.00mm_Horizontal
- J2: renamed from U; value (none) -> Conn_Batt2; footprint (none) -> Connector_JST:JST_PH_S2B-PH-SM4-TB_1x02-1MP_P2.00mm_Horizontal
- J3: renamed from J; value Conn_02x01 -> Conn_Jumper; footprint (none) -> Connector_PinHeader_2.54mm:PinHeader_1x02_P2.54mm_Vertical
Connections:
- net GND: now also H_GND.1, P_GND.1 (Pin_1)
- net at J1.1 (Pin_1), J3.1 (Pin_1): now also H1.1, P1.1 (Pin_1)
- net at J2.1 (Pin_1), J3.2 (Pin_2): now also H2.1, P2.1 (Pin_1)

Commit message: Design updated
Parts:
- renumbered H_GND to H_GND1, P_GND to P_GND1
Changed lines of the file:
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@@
   (symbol (lib_id "Connector:Conn_01x01_Male") (at 110.49 97.79 90) (unit 1)
     (in_bom yes) (on_board yes) (dnp no) (fields_autoplaced)
-    (property "Reference" "P_GND" (at 111.76 95.885 90)
+    (property "Reference" "P_GND1" (at 111.76 95.885 90)
       (effects (font (size 1.27 1.27)) (justify right))
     )
@@
       (project "lipo_disconnector"
         (path "/52cc1f4c-1a58-4a02-bb4f-ffb524d89c3c"
-          (reference "P_GND") (unit 1)
+          (reference "P_GND1") (unit 1)
         )
       )
@@
   (symbol (lib_id "Mechanical:MountingHole_Pad") (at 99.06 95.25 180) (unit 1)
     (in_bom yes) (on_board yes) (dnp no) (fields_autoplaced)
-    (property "Reference" "H_GND" (at 96.52 97.79 0)
+    (property "Reference" "H_GND1" (at 96.52 97.79 0)
       (effects (font (size 1.27 1.27)) (justify left))
     )
@@
       (project "lipo_disconnector"
         (path "/52cc1f4c-1a58-4a02-bb4f-ffb524d89c3c"
-          (reference "H_GND") (unit 1)
+          (reference "H_GND1") (unit 1)
         )
       )
