File: lipo_disconnector.kicad_pcb (KiCad board)
At the start: 2 copper layers, 35 x 10 mm, 13 parts, among them J1 Conn_Batt1, J2 Conn_Batt2, J3 Conn_Jumper

Commit message: update
Parts:
- removed G***: LOGO, Symbols_Extra:SolderParty-New-Logo_3x2.5mm_SilkScreen
- removed kibuzzard-62E1C3A6: G***, kibuzzard-62E1C3A6
- removed kibuzzard-62E1C4AB: G***, kibuzzard-62E1C4AB
- added H1: MountingHole_Pad, MountingHole:MountingHole_4mm_Pad, F.Cu at (151.1, 111.8)
- added H2: MountingHole_Pad, MountingHole:MountingHole_4mm_Pad, F.Cu at (162.6, 111.8)
- added H_GND1: MountingHole_Pad, MountingHole:MountingHole_4mm_Pad, F.Cu at (139.7, 111.8)
- added P1: Conn_01x01_Male, Connector_PinHeader_2.54mm:PinHeader_1x01_P2.54mm_Vertical, F.Cu at (146.1, 108.0)
- added P2: Conn_01x01_Male, Connector_PinHeader_2.54mm:PinHeader_1x01_P2.54mm_Vertical, F.Cu at (157.5, 108.0)
- added P_GND1: Conn_01x01_Male, Connector_PinHeader_2.54mm:PinHeader_1x01_P2.54mm_Vertical, F.Cu at (134.6, 108.0)
Routing:
- net Net-(J1-Pin_1): track 8.69 -> 22.1 mm
- net Net-(J2-Pin_1): track 8.70 -> 21.6 mm
Other:
- board size 35 x 10 mm -> 35 x 21.3 mm
- board text added: "Battery Disco"

Commit message: Design updated
Parts:
- removed H_GND1: MountingHole_Pad, MountingHole:MountingHole_4mm_Pad
- added GND: MountingHole_Pad, MountingHole:MountingHole_4mm_Pad, F.Cu at (149.9, 114.3)
- moved kibuzzard-62E1C2B7 11.2 mm to (167.4, 103.9)
- moved kibuzzard-62E1C2B7 10.9 mm to (167.4, 99.3)
- moved GND 10.2 mm to (144.8, 109.2)
- moved H1 9.25 mm to (160.0, 114.3)
- moved P1 8.98 mm to (154.9, 109.2)
- moved J1 8.33 mm to (146.4, 101.6)
- moved J2 8.33 mm to (171.2, 101.6)
- moved J3 8.33 mm to (157.5, 101.6)
- moved kibuzzard-62E2BF27 8.04 mm to (158.5, 97.9)
- moved kibuzzard-62E2BF3F 8.04 mm to (158.5, 99.6)
- moved kibuzzard-62E2BF4D 8.04 mm to (158.5, 103.4)
- moved H2 8.03 mm to (170.2, 114.3)
- moved P2 7.73 mm to (165.1, 109.2)
- moved kibuzzard-62E1C2B7 5.87 mm to (149.9, 103.9)
- moved kibuzzard-62E1C2B7 5.36 mm to (149.9, 99.3)
- renumbered P_GND1 to GND
Routing:
- net Net-(J1-Pin_1): track 22.1 -> 23.7 mm
- net Net-(J2-Pin_1): track 21.6 -> 22.8 mm
Other:
- board size 35 x 21.3 mm -> 35 x 22.8 mm
- board text added: "J1"
- board text added: "J2"

Commit message: Update lipo_disconnector.kicad_pcb
Parts:
- removed kibuzzard-62E2BF27: G***, kibuzzard-62E2BF27
- removed kibuzzard-62E2BF3F: G***, kibuzzard-62E2BF3F
- removed kibuzzard-62E2BF4D: G***, kibuzzard-62E2BF4D
Other:
- outline, holes or cut-outs redrawn
- board text added: "Always check polarity. Don't cross the streams."
- board text added: "https://opendeved.net/battdisco"
